File: hardware/SliderBar.kicad_pcb (KiCad board)
At the start: 2 copper layers, 50 x 30.1 mm, 35 parts, among them J1 USB_B_Mini, J2 MOTOR, J3 TAPER_RIGHT, J4 TAPER_LEFT, J5 DEBUG, U1 MIC5205-3.3YM5, U2 MT3608, U3 STM32F072C8Tx, U4 TB6612FNG

Commit message: Finished prototype PCB & 3D
Parts:
- moved C11 18.5 mm to (176.4, 58.4)
- moved C13 9.65 mm to (159.0, 70.2), turned to 90 degrees
- moved C3 0.12 mm to (180.3, 77.0)
Connections:
- U3 pad 19: TOUCH_SENSE -> (no net)
- U3 pad 41: (no net) -> TOUCH_SENSE
Routing:
- net +3V3: track 0.00 -> 100.0 mm, vias 0 -> 2
- net +5V: track 0.00 -> 81.0 mm, vias 0 -> 1
- net NRST: track 0.00 -> 60.1 mm
- net +10V: track 0.00 -> 47.8 mm
- net POT: track 0.00 -> 34.4 mm, vias 0 -> 1
- net GND: track 0.00 -> 34.0 mm, vias 0 -> 18
- net SWCLK: track 0.00 -> 25.0 mm, vias 0 -> 2
- net USB_DP: track 0.00 -> 23.1 mm
- net TOUCH_SENSE: track 0.00 -> 22.2 mm, vias 0 -> 1
- net USB_DN: track 0.00 -> 19.2 mm
- net MOT_IN_2: track 0.00 -> 14.7 mm, vias 0 -> 3
- net MOT_IN_1: track 0.00 -> 13.6 mm, vias 0 -> 3
- net Net-(R3-Pad2): track 0.00 -> 12.6 mm
- net STBY: track 0.00 -> 12.4 mm, vias 0 -> 1
- net SWDIO: track 0.00 -> 11.7 mm, vias 0 -> 2
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- added copper zone on B.Cu, net GND
- added copper zone on F.Cu, net GND
Other:
- net class PowerLowVoltage: trace_width 0.4064 -> 0.381
