File: hardware/SliderBar.sch (KiCad schematic (older format))
At the start: 35 parts, among them J1 USB_B_Mini, J2 MOTOR, J3 TAPER_RIGHT, J4 TAPER_LEFT, J5 DEBUG, U1 MIC5205-3.3YM5, U2 MT3608, U3 STM32F072C8Tx, U4 TB6612FNG

Commit message: Placed some components, fixed schematic
Parts:
- R1: footprint Resistor_SMD:R_1206_3216Metric_Pad1.42x1.75mm_HandSolder -> Resistor_SMD:R_0805_2012Metric_Pad1.15x1.40mm_HandSolder
- R2: renamed from R4; footprint Resistor_SMD:R_1206_3216Metric_Pad1.42x1.75mm_HandSolder -> Resistor_SMD:R_0805_2012Metric_Pad1.15x1.40mm_HandSolder
- R3: renamed from R5; footprint Resistor_SMD:R_1206_3216Metric_Pad1.42x1.75mm_HandSolder -> Resistor_SMD:R_0805_2012Metric_Pad1.15x1.40mm_HandSolder
- R4: renamed from R6; footprint Resistor_SMD:R_1206_3216Metric_Pad1.42x1.75mm_HandSolder -> Resistor_SMD:R_0805_2012Metric_Pad1.15x1.40mm_HandSolder
- R5: renamed from R7; footprint Resistor_SMD:R_1206_3216Metric_Pad1.42x1.75mm_HandSolder -> Resistor_SMD:R_0805_2012Metric_Pad1.15x1.40mm_HandSolder
Changed lines of the file:
@@
 $EndComp
 $Comp
-L Device:R R5
+L Device:R R3
 U 1 1 5BC47906
 P 2150 4200
-F 0 "R5" V 2265 4200 50  0000 C CNN
+F 0 "R3" V 2265 4200 50  0000 C CNN
 F 1 "3k" V 2356 4200 50  0000 C CNN
-F 2 "Resistor_SMD:R_1206_3216Metric_Pad1.42x1.75mm_HandSolder" V 2080 4200 50  0001 C CNN
+F 2 "Resistor_SMD:R_0805_2012Metric_Pad1.15x1.40mm_HandSolder" V 2080 4200 50  0001 C CNN
 F 3 "~" H 2150 4200 50  0001 C CNN
 	1    2150 4200
@@
 	3750 1300 3750 1200
 $Comp
-L Device:R R6
+L Device:R R4
 U 1 1 5BDBEFF0
 P 3750 1550
-F 0 "R6" H 3820 1596 50  0000 L CNN
+F 0 "R4" H 3820 1596 50  0000 L CNN
 F 1 "1k" H 3820 1505 50  0000 L CNN
-F 2 "Resistor_SMD:R_1206_3216Metric_Pad1.42x1.75mm_HandSolder" V 3680 1550 50  0001 C CNN
+F 2 "Resistor_SMD:R_0805_2012Metric_Pad1.15x1.40mm_HandSolder" V 3680 1550 50  0001 C CNN
 F 3 "~" H 3750 1550 50  0001 C CNN
 	1    3750 1550
@@
 USB_DP
 $Comp
-L Device:R_Small R4
+L Device:R_Small R2
 U 1 1 5BDD3A19
 P 1750 5600
-F 0 "R4" H 1809 5646 50  0000 L CNN
+F 0 "R2" H 1809 5646 50  0000 L CNN
 F 1 "1.5k" H 1809 5555 50  0000 L CNN
-F 2 "Resistor_SMD:R_1206_3216Metric_Pad1.42x1.75mm_HandSolder" H 1750 5600 50  0001 C CNN
+F 2 "Resistor_SMD:R_0805_2012Metric_Pad1.15x1.40mm_HandSolder" H 1750 5600 50  0001 C CNN
 F 3 "~" H 1750 5600 50  0001 C CNN
 	1    1750 5600
@@
 F 0 "R1" V 1354 6300 50  0000 C CNN
 F 1 "100k" V 1445 6300 50  0000 C CNN
-F 2 "Resistor_SMD:R_1206_3216Metric_Pad1.42x1.75mm_HandSolder" H 1250 6300 50  0001 C CNN
+F 2 "Resistor_SMD:R_0805_2012Metric_Pad1.15x1.40mm_HandSolder" H 1250 6300 50  0001 C CNN
 F 3 "~" H 1250 6300 50  0001 C CNN
 	1    1250 6300
@@
 $EndComp
 $Comp
-L Device:R_Small R7
+L Device:R_Small R5
 U 1 1 5BEDBA2D
 P 5700 3750
-F 0 "R7" H 5641 3796 50  0000 R CNN
+F 0 "R5" H 5641 3796 50  0000 R CNN
 F 1 "10k" H 5641 3705 50  0000 R CNN
-F 2 "Resistor_SMD:R_1206_3216Metric_Pad1.42x1.75mm_HandSolder" H 5700 3750 50  0001 C CNN
+F 2 "Resistor_SMD:R_0805_2012Metric_Pad1.15x1.40mm_HandSolder" H 5700 3750 50  0001 C CNN
 F 3 "~" H 5700 3750 50  0001 C CNN
 	1    5700 3750

Commit message: Finished prototype PCB & 3D
Connections:
- net TOUCH_SENSE: now also U3.41 (PB5); no longer U3.19 (PB1)
Changed lines of the file:
@@
 NoConn ~ 5900 4750
 NoConn ~ 5900 4850
-NoConn ~ 5900 4950
 NoConn ~ 5900 5050
 NoConn ~ 5900 5150
@@
 	2150 3950 2350 3950
 NoConn ~ 2500 4100
-Text GLabel 5900 4550 0    50   Input ~ 0
+Text GLabel 5900 4950 0    50   Input ~ 0
 TOUCH_SENSE
 Wire Wire Line
@@
 Wire Wire Line
 	1350 5900 1850 5900
+NoConn ~ 5900 4550
 $EndSCHEMATC
