File: hardware_old/SliderBar.sch (KiCad schematic (older format))
At the start: 35 parts, among them J1 USB_B_Mini, J2 MOTOR, J3 TAPER_RIGHT, J4 TAPER_LEFT, J5 DEBUG, U1 MIC5205-3.3YM5, U2 MT3608, U3 STM32F072C8Tx, U4 TB6612FNG

Commit message: Add STM32F072C8 MCU
Parts:
- D1, D2, D3: symbol nelib:STPS1L40 -> SliderBar-rescue:STPS1L40-nelib
- U2: symbol nelib:MT3608 -> SliderBar-rescue:MT3608-nelib
Changed lines of the file:
@@
 NRST
 $Comp
-L power:GND #PWR?
+L power:GND #PWR019
 U 1 1 5BB23C60
 P 4000 4650
-F 0 "#PWR?" H 4000 4400 50  0001 C CNN
+F 0 "#PWR019" H 4000 4400 50  0001 C CNN
 F 1 "GND" V 4000 4500 50  0000 R CNN
 F 2 "" H 4000 4650 50  0001 C CNN
@@
 POT
 $Comp
-L power:GND #PWR?
+L power:GND #PWR018
 U 1 1 5BB24025
 P 4000 4100
-F 0 "#PWR?" H 4000 3850 50  0001 C CNN
+F 0 "#PWR018" H 4000 3850 50  0001 C CNN
 F 1 "GND" H 4005 3927 50  0000 C CNN
 F 2 "" H 4000 4100 50  0001 C CNN
@@
 $EndComp
 $Comp
-L power:+3.3V #PWR?
+L power:+3.3V #PWR017
 U 1 1 5BB24078
 P 4000 3550
-F 0 "#PWR?" H 4000 3400 50  0001 C CNN
+F 0 "#PWR017" H 4000 3400 50  0001 C CNN
 F 1 "+3.3V" H 4015 3723 50  0000 C CNN
 F 2 "" H 4000 3550 50  0001 C CNN
@@
 $EndComp
 $Comp
-L power:GND #PWR?
+L power:GND #PWR030
 U 1 1 5BB24638
 P 9350 6050
-F 0 "#PWR?" H 9350 5800 50  0001 C CNN
+F 0 "#PWR030" H 9350 5800 50  0001 C CNN
 F 1 "GND" H 9355 5877 50  0000 C CNN
 F 2 "" H 9350 6050 50  0001 C CNN
@@
 MOT_IN_PWM
 $Comp
-L power:+10V #PWR?
+L power:+10V #PWR031
 U 1 1 5BB2664B
 P 9950 3450
-F 0 "#PWR?" H 9950 3300 50  0001 C CNN
+F 0 "#PWR031" H 9950 3300 50  0001 C CNN
 F 1 "+10V" H 9965 3623 50  0000 C CNN
 F 2 "" H 9950 3450 50  0001 C CNN
@@
 	9750 3900 9750 3950
 $Comp
-L power:+3V3 #PWR?
+L power:+3V3 #PWR029
 U 1 1 5BB27786
 P 9350 3950
-F 0 "#PWR?" H 9350 3800 50  0001 C CNN
+F 0 "#PWR029" H 9350 3800 50  0001 C CNN
 F 1 "+3V3" H 9300 4100 50  0000 C CNN
 F 2 "" H 9350 3950 50  0001 C CNN
@@
 MOT_IN_2
 $Comp
-L power:GND #PWR?
+L power:GND #PWR032
 U 1 1 5BB27E3D
 P 10400 4000
-F 0 "#PWR?" H 10400 3750 50  0001 C CNN
+F 0 "#PWR032" H 10400 3750 50  0001 C CNN
 F 1 "GND" V 10405 3872 50  0000 R CNN
 F 2 "" H 10400 4000 50  0001 C CNN
@@
 Connection ~ 9950 3900
 $Comp
-L power:+3V3 #PWR?
+L power:+3V3 #PWR026
 U 1 1 5BCA2B2D
 P 6600 2950
-F 0 "#PWR?" H 6600 2800 50  0001 C CNN
+F 0 "#PWR026" H 6600 2800 50  0001 C CNN
 F 1 "+3V3" H 6615 3123 50  0000 C CNN
 F 2 "" H 6600 2950 50  0001 C CNN
@@
 Connection ~ 6500 3050
 $Comp
-L power:GND #PWR?
+L power:GND #PWR025
 U 1 1 5BCAB682
 P 6400 6350
-F 0 "#PWR?" H 6400 6100 50  0001 C CNN
+F 0 "#PWR025" H 6400 6100 50  0001 C CNN
 F 1 "GND" H 6405 6177 50  0000 C CNN
 F 2 "" H 6400 6350 50  0001 C CNN
@@
 Connection ~ 6700 3050
 $Comp
-L power:GND #PWR?
+L power:GND #PWR023
 U 1 1 5BCB754A
 P 5350 3750
-F 0 "#PWR?" H 5350 3500 50  0001 C CNN
+F 0 "#PWR023" H 5350 3500 50  0001 C CNN
 F 1 "GND" H 5355 3577 50  0000 C CNN
 F 2 "" H 5350 3750 50  0001 C CNN
@@
 	2050 1800 2050 1700
 $Comp
-L power:GND #PWR?
+L power:GND #PWR09
 U 1 1 5BD40D38
 P 2050 1800
-F 0 "#PWR?" H 2050 1550 50  0001 C CNN
+F 0 "#PWR09" H 2050 1550 50  0001 C CNN
 F 1 "GND" H 2055 1627 50  0000 C CNN
 F 2 "" H 2050 1800 50  0001 C CNN
@@
 $EndComp
 $Comp
-L power:+3V3 #PWR?
+L power:+3V3 #PWR08
 U 1 1 5BCA296C
 P 1900 1200
-F 0 "#PWR?" H 1900 1050 50  0001 C CNN
+F 0 "#PWR08" H 1900 1050 50  0001 C CNN
 F 1 "+3V3" H 1915 1373 50  0000 C CNN
 F 2 "" H 1900 1200 50  0001 C CNN
@@
 3.3V REGULATOR
 $Comp
-L power:GND #PWR?
+L power:GND #PWR06
 U 1 1 5BC34408
 P 1500 2000
-F 0 "#PWR?" H 1500 1750 50  0001 C CNN
+F 0 "#PWR06" H 1500 1750 50  0001 C CNN
 F 1 "GND" H 1505 1827 50  0000 C CNN
 F 2 "" H 1500 2000 50  0001 C CNN
@@
 Id = sqrt(Iout * Imax)
 $Comp
-L power:GND #PWR?
+L power:GND #PWR012
 U 1 1 5BC4D897
 P 2850 3850
-F 0 "#PWR?" H 2850 3600 50  0001 C CNN
+F 0 "#PWR012" H 2850 3600 50  0001 C CNN
 F 1 "GND" H 2855 3677 50  0000 C CNN
 F 2 "" H 2850 3850 50  0001 C CNN
@@
 Recommended:\n4.7uH - 22uH
 $Comp
-L power:GND #PWR?
+L power:GND #PWR010
 U 1 1 5BC48783
 P 2150 4450
-F 0 "#PWR?" H 2150 4200 50  0001 C CNN
+F 0 "#PWR010" H 2150 4200 50  0001 C CNN
 F 1 "GND" H 2155 4277 50  0000 C CNN
 F 2 "" H 2150 4450 50  0001 C CNN
@@
 $EndComp
 $Comp
-L power:+10V #PWR?
+L power:+10V #PWR011
 U 1 1 5BC3AC64
 P 2850 3250
-F 0 "#PWR?" H 2850 3100 50  0001 C CNN
+F 0 "#PWR011" H 2850 3100 50  0001 C CNN
 F 1 "+10V" H 2865 3423 50  0000 C CNN
 F 2 "" H 2850 3250 50  0001 C CNN
@@
 $EndComp
 $Comp
-L power:GND #PWR?
+L power:GND #PWR02
 U 1 1 5BC3A8CB
 P 900 4050
-F 0 "#PWR?" H 900 3800 50  0001 C CNN
+F 0 "#PWR02" H 900 3800 50  0001 C CNN
 F 1 "GND" H 905 3877 50  0000 C CNN
 F 2 "" H 900 4050 50  0001 C CNN
@@
 $EndComp
 $Comp
-L nelib:MT3608 U2
+L SliderBar-rescue:MT3608-nelib U2
 U 1 1 5BC394FC
 P 1650 3850
@@
 Connection ~ 9950 3550
 $Comp
-L power:+5V #PWR?
+L power:+5V #PWR04
 U 1 1 5BD9F21E
 P 1100 1200
-F 0 "#PWR?" H 1100 1050 50  0001 C CNN
+F 0 "#PWR04" H 1100 1050 50  0001 C CNN
 F 1 "+5V" H 1115 1373 50  0000 C CNN
 F 2 "" H 1100 1200 50  0001 C CNN
@@
 $EndComp
 $Comp
-L power:+5V #PWR?
+L power:+5V #PWR01
 U 1 1 5BD9F4E9
 P 900 3250
-F 0 "#PWR?" H 900 3100 50  0001 C CNN
+F 0 "#PWR01" H 900 3100 50  0001 C CNN
 F 1 "+5V" H 915 3423 50  0000 C CNN
 F 2 "" H 900 3250 50  0001 C CNN
@@
 $EndComp
 $Comp
-L power:VBUS #PWR?
+L power:VBUS #PWR013
 U 1 1 5BD9F98D
 P 3000 1300
-F 0 "#PWR?" H 3000 1150 50  0001 C CNN
+F 0 "#PWR013" H 3000 1150 50  0001 C CNN
 F 1 "VBUS" H 3015 1473 50  0000 C CNN
 F 2 "" H 3000 1300 50  0001 C CNN
@@
 $EndComp
 $Comp
-L power:+5V #PWR?
+L power:+5V #PWR015
 U 1 1 5BD9FC3F
 P 3750 1200
-F 0 "#PWR?" H 3750 1050 50  0001 C CNN
+F 0 "#PWR015" H 3750 1050 50  0001 C CNN
 F 1 "+5V" H 3765 1373 50  0000 C CNN
 F 2 "" H 3750 1200 50  0001 C CNN
@@
 $EndComp
 $Comp
-L power:GND #PWR?
+L power:GND #PWR016
 U 1 1 5BDBF2FB
 P 3750 2200
-F 0 "#PWR?" H 3750 1950 50  0001 C CNN
+F 0 "#PWR016" H 3750 1950 50  0001 C CNN
 F 1 "GND" H 3755 2027 50  0000 C CNN
 F 2 "" H 3750 2200 50  0001 C CNN
@@
 USB_DP
 $Comp
-L power:GND #PWR?
+L power:GND #PWR03
 U 1 1 5BDDF695
 P 950 6400
-F 0 "#PWR?" H 950 6150 50  0001 C CNN
+F 0 "#PWR03" H 950 6150 50  0001 C CNN
 F 1 "GND" H 955 6227 50  0000 C CNN
 F 2 "" H 950 6400 50  0001 C CNN
@@
 Connection ~ 10400 3900
 $Comp
-L power:VPP #PWR?
+L power:VPP #PWR020
 U 1 1 5BD8AB17
 P 4000 4850
-F 0 "#PWR?" H 4000 4700 50  0001 C CNN
+F 0 "#PWR020" H 4000 4700 50  0001 C CNN
 F 1 "VPP" V 4000 5150 50  0000 R CNN
 F 2 "" H 4000 4850 50  0001 C CNN
@@
 $EndComp
 $Comp
-L power:VPP #PWR?
+L power:VPP #PWR014
 U 1 1 5BD8AD8C
 P 3000 1650
-F 0 "#PWR?" H 3000 1500 50  0001 C CNN
+F 0 "#PWR014" H 3000 1500 50  0001 C CNN
 F 1 "VPP" H 3015 1823 50  0000 C CNN
 F 2 "" H 3000 1650 50  0001 C CNN
@@
 CONNECTORS
 $Comp
-L power:VBUS #PWR?
+L power:VBUS #PWR05
 U 1 1 5BE0AEED
 P 1450 5500
-F 0 "#PWR?" H 1450 5350 50  0001 C CNN
+F 0 "#PWR05" H 1450 5350 50  0001 C CNN
 F 1 "VBUS" H 1465 5673 50  0000 C CNN
 F 2 "" H 1450 5500 50  0001 C CNN
@@
 Connection ~ 1050 6300
 $Comp
-L power:+3V3 #PWR?
+L power:+3V3 #PWR07
 U 1 1 5BE2449C
 P 1750 5400
-F 0 "#PWR?" H 1750 5250 50  0001 C CNN
+F 0 "#PWR07" H 1750 5250 50  0001 C CNN
 F 1 "+3V3" H 1765 5573 50  0000 C CNN
 F 2 "" H 1750 5400 50  0001 C CNN
@@
 	10900 2950 10900 6300
 $Comp
-L power:+3V3 #PWR?
+L power:+3V3 #PWR021
 U 1 1 5BE61DFB
 P 4950 1200
-F 0 "#PWR?" H 4950 1050 50  0001 C CNN
+F 0 "#PWR021" H 4950 1050 50  0001 C CNN
 F 1 "+3V3" H 4965 1373 50  0000 C CNN
 F 2 "" H 4950 1200 50  0001 C CNN
@@
 $EndComp
 $Comp
-L power:GND #PWR?
+L power:GND #PWR022
 U 1 1 5BE61E6A
 P 4950 1800
-F 0 "#PWR?" H 4950 1550 50  0001 C CNN
+F 0 "#PWR022" H 4950 1550 50  0001 C CNN
 F 1 "GND" H 4955 1627 50  0000 C CNN
 F 2 "" H 4950 1800 50  0001 C CNN
@@
 $EndComp
 $Comp
-L power:GND #PWR?
+L power:GND #PWR028
 U 1 1 5BE61EC4
 P 6700 1800
-F 0 "#PWR?" H 6700 1550 50  0001 C CNN
+F 0 "#PWR028" H 6700 1550 50  0001 C CNN
 F 1 "GND" H 6705 1627 50  0000 C CNN
 F 2 "" H 6700 1800 50  0001 C CNN
@@
 $EndComp
 $Comp
-L power:+5V #PWR?
+L power:+5V #PWR027
 U 1 1 5BE6210E
 P 6700 1200
-F 0 "#PWR?" H 6700 1050 50  0001 C CNN
+F 0 "#PWR027" H 6700 1050 50  0001 C CNN
 F 1 "+5V" H 6715 1373 50  0000 C CNN
 F 2 "" H 6700 1200 50  0001 C CNN
@@
 	6700 1400 6700 1200
 $Comp
-L power:GND #PWR?
+L power:GND #PWR024
 U 1 1 5BEDB912
 P 5700 3950
-F 0 "#PWR?" H 5700 3700 50  0001 C CNN
+F 0 "#PWR024" H 5700 3700 50  0001 C CNN
 F 1 "GND" H 5705 3777 50  0000 C CNN
 F 2 "" H 5700 3950 50  0001 C CNN
@@
 	3400 5100 4800 5100
 $Comp
-L nelib:STPS1L40 D2
+L SliderBar-rescue:STPS1L40-nelib D2
 U 1 1 5C4BAB9A
 P 3300 1300
@@
 $EndComp
 $Comp
-L nelib:STPS1L40 D3
+L SliderBar-rescue:STPS1L40-nelib D3
 U 1 1 5C4C2FBE
 P 3300 1650
@@
 $EndComp
 $Comp
-L nelib:STPS1L40 D1
+L SliderBar-rescue:STPS1L40-nelib D1
 U 1 1 5C4C4325
 P 2350 3350
